Commit message: 

File: urdf/sr_hand_vm_compatible.urdf (robot description, URDF)
Before this commit: robot shadowhand_motor, 33 links, 32 joints
Links:
- link rh_ffdistal: geometry collision mesh filename=package://sr_description_vmc/meshes/components/f_distal/pst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; visual mesh filename=package://sr_description_vmc/meshes/components/f_distal/pst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
- link rh_ffknuckle: geometry collision cylinder length=0.014 radius=0.007; visual mesh filename=package://sr_description_vmc/meshes/components/f_knuckle/f_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
- link rh_ffmiddle: geometry collision cylinder length=0.025 radius=0.007; collision sphere radius=0.007
- link rh_ffproximal: geometry collision cylinder length=0.040 radius=0.007; visual mesh filename=package://sr_description_vmc/meshes/components/f_proximal/f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
- link rh_forearm: geometry collision box size=0.07 0.07 0.07; collision mesh filename=package://sr_description_vmc/meshes/components/forearm/fore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
- link rh_lfdistal: geometry collision mesh filename=package://sr_description_vmc/meshes/components/f_distal/pst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; visual mesh filename=package://sr_description_vmc/meshes/components/f_distal/pst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
- link rh_lfknuckle: geometry collision cylinder length=0.014 radius=0.007; visual mesh filename=package://sr_description_vmc/meshes/components/f_knuckle/f_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
- link rh_lfmetacarpal: geometry collision box size=0.018 0.024 0.040; visual mesh filename=package://sr_description_vmc/meshes/components/lf_metacarpa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
- link rh_lfmiddle: geometry collision cylinder length=0.025 radius=0.007; collision sphere radius=0.007
- link rh_lfproximal: geometry collision cylinder length=0.040 radius=0.007; visual mesh filename=package://sr_description_vmc/meshes/components/f_proximal/f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
- link rh_mfdistal: geometry collision mesh filename=package://sr_description_vmc/meshes/components/f_distal/pst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; visual mesh filename=package://sr_description_vmc/meshes/components/f_distal/pst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
- link rh_mfknuckle: geometry collision cylinder length=0.014 radius=0.007; visual mesh filename=package://sr_description_vmc/meshes/components/f_knuckle/f_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
- link rh_mfmiddle: geometry collision cylinder length=0.025 radius=0.007; collision sphere radius=0.007
- link rh_mfproximal: geometry collision cylinder length=0.040 radius=0.007; visual mesh filename=package://sr_description_vmc/meshes/components/f_proximal/f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
- link rh_palm: geometry collision box size=0.018 0.024 0.004; collision box size=0.020 0.024 0.040
- link rh_rfdistal: geometry collision mesh filename=package://sr_description_vmc/meshes/components/f_distal/pst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; visual mesh filename=package://sr_description_vmc/meshes/components/f_distal/pst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
- link rh_rfknuckle: geometry collision cylinder length=0.014 radius=0.007; visual mesh filename=package://sr_description_vmc/meshes/components/f_knuckle/f_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
- link rh_rfmiddle: geometry collision cylinder length=0.025 radius=0.007; collision sphere radius=0.007
- link rh_rfproximal: geometry collision cylinder length=0.040 radius=0.007; visual mesh filename=package://sr_description_vmc/meshes/components/f_proximal/f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
- link rh_thdistal: geometry collision mesh filename=package://sr_description_vmc/meshes/components/th_distal/ps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; visual mesh filename=package://sr_description_vmc/meshes/components/th_distal/ps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
- link rh_thmiddle: geometry collision cylinder length=0.014 radius=0.010; collision cylinder length=0.018 radius=0.011
- link rh_thproximal: geometry collision cylinder length=0.018 radius=0.012; visual mesh filename=package://sr_description_vmc/meshes/components/th_proximal/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
- link rh_wrist: geometry collision box size=0.027 0.018 0.010; collision box size=0.027 0.018 0.010
